Commit message: feat(worx): ros2_control hardware interface for the Worx mainboard
WorxSystem talks to the Worx board firmware over SPI with its existing
JSON protocol (fixed 250-byte transfers, SOF/EOF framing, ping watchdog),
so the firmware needs no change. Layers:

- worx_protocol: framing + commands (key order as in the ROS1 worx_comms)
  + status parsing, checked against real lines from the robot's logs
  (MotorPulse Emergancy/BlockForward, MotorCurrent Mow, powerState).
- WheelOdometer: cumulative tick magnitude + direction bit -> distance,
  with wrap and glitch guards.
- WorxLink: 1 ms SPI loop thread; spidev transport or a fake board that
  emulates the firmware for tests and bench runs.
- WorxSystem: wheels (velocity cmd, position/velocity state, open-loop
  PWM like worx_comms), blade (effort 0..1 -> mow PWM), /power,
  /power/charger_present (InCharger), /worx/status, /worx/emergency,
  /worx/motors_enabled. The blade stays off after emergency/link loss until
  commanded off once, and stops after 25 s without drive commands.

Hardware selection: OM_HARDWARE=worx picks config/hardware/worx.yaml and
the Worx ros2_control block; micro-ROS agent is skipped for Worx. Adds
hardware_bench.launch.py (drive stack only) and fixes the controller
manager to take robot_description from the topic (Jazzy ignores the param).

Tested: 10 link tests; bench launch in Jazzy with the fake board (drive,
turn, blade, emergency, idle timeout).

Co-Authored-By: Claude Opus 5.5 <noreply@anthropic.com>

File: description/robot.urdf.xacro (robot description, xacro)
@@ -3,5 +3,9 @@
     <xacro:arg name="use_ros2_control" default="true"/>
     <xacro:arg name="sim_mode" default="false"/>
-    <xacro:property name="robot_yaml" value="$(find open_mower_next)/config/hardware/yardforce500.yaml" />
+    <!-- config/hardware/<hardware>.yaml; "worx" selects the Worx mainboard plugin -->
+    <xacro:arg name="hardware" default="yardforce500"/>
+    <xacro:arg name="worx_transport" default="spidev"/>
+    <xacro:property name="hardware" value="$(arg hardware)"/>
+    <xacro:property name="robot_yaml" value="$(find open_mower_next)/config/hardware/${hardware}.yaml" />
     <xacro:property name="robot" value="${xacro.load_yaml(robot_yaml)}"/>
     <xacro:include filename="robot_core.xacro" />

File: description/ros2_control.xacro (robot description, xacro)
@@ -1,5 +1,8 @@
 <?xml version="1.0"?>
 <robot xmlns:xacro="http://www.ros.org/wiki/xacro">
-    <xacro:unless value="$(arg sim_mode)">
+    <xacro:if value="${hardware == 'worx' and '$(arg sim_mode)' != 'true'}">
+        <xacro:include filename="ros2_control_worx.xacro" />
+    </xacro:if>
+    <xacro:unless value="${'$(arg sim_mode)' == 'true' or hardware == 'worx'}">
         <xacro:property name="vesc_yaml" value="$(find open_mower_next)/config/hardware/vesc.yaml" />
         <xacro:property name="vesc" value="${xacro.load_yaml(vesc_yaml)}"/>
